File: schematic/prot/Init_prot.kicad_sch (KiCad schematic)
At the start: 19 parts, among them J1 Conn_01x02, J2 Contactor, J3 FC, Q1 AO3400A, SW1 SW_DIP_x01, U1 STM32F070F6Px, U2 MPU-6050

Commit message: Schematic update
Parts:
- added C10, C4: 0.1u, symbol Device:C
- added C3: 1000u, symbol Device:C
- added C7, C8: 22u, symbol Device:C
- added C9: 10u, symbol Device:C
- added J4: Conn_01x06_Pin, symbol Connector:Conn_01x06_Pin
- added L1: 10u, symbol Device:L
- added R10: 510k, symbol Device:R
- added R11, R8: 100k, symbol Device:R
- added R9: 22k, symbol Device:R
- added U3: TPS54302, Package_TO_SOT_SMD:SOT-23-6, symbol Regulator_Switching:TPS54302
Connections:
- net +24V: now also C10.2, C3.1, C9.2, R10.1, U3.3 (VIN)
- net +3.3V: now also C7.2, C8.2, J4.5 (Pin_5), L1.2, R8.1; no longer D1.4 (BA), D1.5 (GA), D1.6 (RA)
- net FCU INIT: now also J3.2 (Pin_2)
- net GND: now also R4.2, R5.2, R6.2, C10.1, C7.1, C8.1, C9.1, J4.6 (Pin_6), R11.2, R9.2, U3.1 (GND)
- net LED B: now also D1.4 (BA)
- net LED G: now also D1.5 (GA)
- net LED R: now also D1.6 (RA)
- net MPU INIT: now also U2.12 (INT)
- net RX: now also J4.2 (Pin_2)
- net SCL: now also R1.2, U2.23 (SCL)
- net SDA: now also R2.2, U2.24 (SDA)
- net SWCLK: now also J4.3 (Pin_3)
- net SWDIO: now also J4.4 (Pin_4)
- net TX: now also J4.1 (Pin_1)
- net INIT OUT: now reaches Q1.1 (G), R3.1
- net INIT OUT: now also U1.9 (PA3)
- net at J1.1 (Pin_1), Q1.3 (D): now also C3.2
- net Logic IN: now reaches J2.2 (Pin_2)
- net Logic IN: now also U1.8 (PA2)
- new net: C4.1, L1.1, U3.2 (SW)
- new net: C4.2, U3.6 (BOOT)
- new net: R10.2, R11.1, U3.5 (EN)
- new net: R8.2, R9.1, U3.4 (FB)
- no-connect marks 3 -> 5
Other:
- moved on the sheet: C1, C2, C5, C6, D1, J1, J2, J3, Q1, R1, R2, R3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
