File: schematic/prot/Init_prot.kicad_sch (KiCad schematic)
At the start: 32 parts, among them J1 Conn_01x02, J2 Contactor, J3 FC, J4 Conn_01x06_Pin, Q1 AO3400A, SW1 SW_DIP_x01, U1 STM32F070F6Px, U2 MPU-6050, U3 TPS54302

Commit message: Schematic
Parts:
- added SW2: SW_DIP_x01, symbol Switch:SW_DIP_x01
- J3: value FC -> FCU
Connections:
- net +24V: no longer R10.1
- net FCU INIT: no longer U1.7 (PA1)
- net GND: now also SW2.1
- net at R11.1, U3.5 (EN): now also R10.1; no longer R10.2
- net Logic IN renamed Contactor INIT
- net Contactor INIT: now also U1.7 (PA1); no longer U1.8 (PA2)
- new net: R10.2, SW2.2
- new net FCU Init: U1.8 (PA2)
Other:
- moved on the sheet: R10, R11

Commit message: Schematic update
Parts:
- added C11: 100n, Capacitor_SMD:C_0805_2012Metric_Pad1.18x1.45mm_HandSolder, symbol Device:C
Connections:
- net +24V: now also SW2.2
- net +3.3V: now also C11.1
- net GND: now also C11.2; no longer SW2.1
- net at R10.2: now also SW2.1; no longer SW2.2
Other:
- moved on the sheet: J2, J3, SW2
