File: schematic/prot/_autosave-Init_prot.kicad_sch (KiCad schematic)
At the start: 32 parts, among them J1 Conn_01x02, J2 Contactor, J3 FC, J4 Conn_01x06_Pin, Q1 AO3400A, SW1 SW_DIP_x01, U1 STM32F070F6Px, U2 MPU-6050, U3 TPS54302

Commit message: Schematic update + GPIO shuffle + MPU/Contactor/FCU INT
Parts:
- J3: value FC -> FCU
Connections:
- net FCU INIT: no longer U1.7 (PA1)
- net Logic IN renamed Contactor INIT
- net Contactor INIT: now also U1.7 (PA1); no longer U1.8 (PA2)
- new net FCU Init: U1.8 (PA2)
Changed lines of the file:
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@@
 			)
 		)
-		(property "Value" "Logic IN"
-			(at 190.5 62.23 0)
-			(effects
-				(font
-					(size 1.27 1.27)
-				)
+		(property "Value" "Contactor INIT"
+			(at 193.04 58.4199 0)
+			(effects
+				(font
+					(size 1.27 1.27)
+				)
+				(justify right)
 			)
 		)
@@
 			)
 		)
-		(property "Value" "FC"
+		(property "Value" "FCU"
 			(at 212.09 26.6699 90)
 			(effects
@@
 			)
 		)
-		(property "Value" "FCU INIT"
+		(property "Value" "Contactor INIT"
 			(at 107.95 96.5199 90)
 			(effects
@@
 			)
 		)
-		(property "Value" "Logic IN"
+		(property "Value" "FCU Init"
 			(at 107.95 99.0599 90)
 			(effects
