File: schematic/SuperCap_version/Init_Supercap_Prot/Init_Supercap_Prot.kicad_sch (KiCad schematic)
At the start: 35 parts, among them J1 Load, J2 Contactor, J3 FCU, J4 Conn_01x06_Pin, J5 Power, Q1 AO3400A, SW1 SW_DIP_x01, SW2 SW_DIP_x01, U1 STM32F070F6Px, U2 MPU-6050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

Commit message: Schematic + BOM
Parts:
- removed C10: 0.1u, symbol Device:C
- removed C7, C8: 22u, symbol Device:C
- removed C9: 10u, symbol Device:C
- removed L1: 10u, symbol Device:L
- removed R10: 510k, symbol Device:R
- removed R11: 100k, symbol Device:R
- removed SW2: SW_DIP_x01, symbol Switch:SW_DIP_x01
- removed U3: TPS54302, Package_TO_SOT_SMD:SOT-23-6, symbol Regulator_Switching:TPS54302
- added BT1: LiPo-1S, symbol Device:Battery
- added D2: LED, symbol Device:LED
- added U3: XC6206PxxxMR, Package_TO_SOT_SMD:SOT-23-3, symbol Regulator_Linear:XC6206PxxxMR
- added U4: MCP73831-2-OT, Package_TO_SOT_SMD:SOT-23-5, symbol Battery_Management:MCP73831-2-OT
- C3: value 1000u -> 4.7u
- C4: value 0.1u -> 100u
- R8: value 100k -> 470R
- R9: value 22k -> 2k; footprint (none) -> Resistor_SMD:R_0805_2012Metric_Pad1.20x1.40mm_HandSolder
Connections:
- net +3.3V: now also U3.2 (VO); no longer R8.1
- net GND: now also C3.2, C4.2, R8.1, BT1.2 (-), U3.1 (GND), U4.2 (V_{SS}); no longer C3.1
- net VBAT: now reaches C4.1
- net VBAT: now also C3.1, J1.2 (Pin_2), BT1.1 (+), U3.3 (VI), U4.3 (V_{BAT})
- net at R8.2: now also D2.1 (K); no longer R9.1
- removed net +24V: C3.2, J1.2 (Pin_2), J5.2 (Pin_2)
- new net: D2.2 (A), U4.1 (STAT)
- new net: R9.1, U4.5 (PROG)
- new net +5V: J5.2 (Pin_2), U4.4 (V_{DD})
Other:
- moved on the sheet: C1, C11, C2, C5, C6, D1, J1, J2, J3, J4, J5, Q1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
